Commit message: update imu param

File: description/imu.xacro (robot description, xacro)
@@ -6,7 +6,7 @@
         <origin xyz="${xyz}" rpy="${rpy}"/>
         <parent link="${parent}"/>
-        <child link="imu_sensor_link"/>
+        <child link="camera_imu_optical_frame"/>
     </joint>
-    <link name="imu_sensor_link">
+    <link name="camera_imu_optical_frame">
         <collision>
             <origin xyz="0 0 0" rpy="0 0 0"/>
@@ -28,5 +28,5 @@
         </inertial>
     </link>
-    <gazebo reference="imu_sensor_link">
+    <!-- <gazebo reference="imu_sensor_link">
         <gravity>true</gravity>
         <sensor name='imu_sensor' type='imu'>
@@ -45,6 +45,6 @@
             <pose>0 0 0 0 0 0</pose>
         </sensor>
-    </gazebo>
+    </gazebo> -->
 </xacro:macro>
-<xacro:imu_sensor xyz="0 0 0" rpy = "0 0 0" parent="base_link" />
+<xacro:imu_sensor xyz="0 0 0" rpy = "0 0 0" parent="camera_link" />
 </robot>

File: description/robot.urdf.xacro (robot description, xacro)
@@ -4,5 +4,5 @@
     <xacro:arg name="sim_mode" default="false"/>
     <xacro:include filename="robot_core.xacro" />
-    <!-- <xacro:include filename="imu.xacro" /> -->
+    <xacro:include filename="imu.xacro" />
     <xacro:if value="$(arg use_ros2_control)">
         <xacro:include filename="ros2_control.xacro" />
