Commit message: update param of wheels

File: description/gazebo_control.xacro (robot description, xacro)
@@ -9,5 +9,5 @@
             <left_joint>left_wheel_joint</left_joint>
             <right_joint>right_wheel_joint</right_joint>
-            <wheel_separation>0.337</wheel_separation>
+            <wheel_separation>0.3366</wheel_separation>
             <wheel_diameter>0.065</wheel_diameter>
             <!-- Limits -->

File: description/robot_core.xacro (robot description, xacro)
@@ -6,9 +6,9 @@
     <xacro:property name="chassis_height" value="0.072"/>
     <xacro:property name="chassis_mass" value="3.0"/>
-    <xacro:property name="wheel_radius" value="0.0325"/>
+    <xacro:property name="wheel_radius" value="0.03185"/>
     <xacro:property name="wheel_thickness" value="0.0255"/>
     <xacro:property name="wheel_mass" value="0.05"/>
     <xacro:property name="wheel_offset_x" value="0.0"/>
-    <xacro:property name="wheel_offset_y" value="0.1685"/>
+    <xacro:property name="wheel_offset_y" value="0.164"/>
     <xacro:property name="wheel_offset_z" value="${-chassis_height+wheel_radius}"/>
     <xacro:property name="caster_wheel_radius" value="0.02"/>
