Commit message: update parameters

File: description/camera.xacro (robot description, xacro)
@@ -4,5 +4,5 @@
         <parent link="chassis"/>
         <child link="camera_link"/>
-        <origin xyz="0.0275 0 0.498" rpy="0 0 0"/>
+        <origin xyz="0.0275 0 0.698" rpy="0 0 0"/>
     </joint>
     <link name="camera_link">

File: description/depth_camera.xacro (robot description, xacro)
@@ -4,5 +4,5 @@
         <parent link="chassis"/>
         <child link="camera_link"/>
-        <origin xyz="0.0275 0 0.498" rpy="0 0 0"/>
+        <origin xyz="0.0275 0 0.698" rpy="0 0 0"/>
     </joint>
     <link name="camera_link">

File: description/lidar.xacro (robot description, xacro)
@@ -4,5 +4,5 @@
         <parent link="chassis"/>
         <child link="laser_frame"/>
-        <origin xyz="-0.02 0 0.5" rpy="0 0 0"/>
+        <origin xyz="-0.02 0 0.7" rpy="0 0 0"/>
     </joint>
     <link name="laser_frame">

File: description/robot_core.xacro (robot description, xacro)
@@ -4,6 +4,5 @@
     <xacro:property name="chassis_radius" value="0.20"/>
     <xacro:property name="chassis_length" value="0.112"/>
-    <!-- <xacro:property name="chassis_width" value="0.265"/> -->
-    <!-- <xacro:property name="chassis_length" value="0.112"/> -->
+    <xacro:property name="chassis_width" value="0.265"/>
     <xacro:property name="chassis_height" value="0.08"/>
     <xacro:property name="chassis_mass" value="1.0"/>
@@ -59,5 +58,5 @@
         </visual>
         <collision>
-            <origin xyz = "0 0 ${chassis_length}/2"/>
+            <origin xyz = "0 0 ${chassis_length/2}"/>
             <geometry>
                 <cylinder length="${chassis_length}" radius="${chassis_radius}"/>
@@ -65,5 +64,5 @@
         </collision>
         <xacro:inertial_cylinder mass="${chassis_mass}" length="${chassis_length}" radius="${chassis_radius}">
-            <origin xyz="0 0 ${chassis_length}/2" rpy="0 0 0"/>
+            <origin xyz="0 0 ${chassis_length/2}" rpy="0 0 0"/>
         </xacro:inertial_cylinder>
     </link>

Commit message: just change something parameters of coordinates

File: description/camera.xacro (robot description, xacro)
@@ -4,5 +4,5 @@
         <parent link="chassis"/>
         <child link="camera_link"/>
-        <origin xyz="0.0275 0 0.698" rpy="0 0 0"/>
+        <origin xyz="0.0275 0 0.6" rpy="0 0 0"/>
     </joint>
     <link name="camera_link">

File: description/depth_camera.xacro (robot description, xacro)
@@ -4,5 +4,5 @@
         <parent link="chassis"/>
         <child link="camera_link"/>
-        <origin xyz="0.0275 0 0.698" rpy="0 0 0"/>
+        <origin xyz="0.0275 0 0.6" rpy="0 0 0"/>
     </joint>
     <link name="camera_link">

File: description/lidar.xacro (robot description, xacro)
@@ -2,7 +2,7 @@
 <robot xmlns:xacro="http://www.ros.org/wiki/xacro" >
     <joint name="laser_joint" type="fixed">
-        <parent link="chassis"/>
+        <parent link="camera_link"/>
         <child link="laser_frame"/>
-        <origin xyz="-0.02 0 0.7" rpy="0 0 0"/>
+        <origin xyz="-0.0475 0 0.022" rpy="0 0 0"/>
     </joint>
     <link name="laser_frame">

Commit message: update params

File: description/camera.xacro (robot description, xacro)
@@ -4,5 +4,5 @@
         <parent link="chassis"/>
         <child link="camera_link"/>
-        <origin xyz="0.0275 0 0.698" rpy="0 0 0"/>
+        <origin xyz="0.042 0 0.583" rpy="0 0 0"/>
     </joint>
     <link name="camera_link">

File: description/depth_camera.xacro (robot description, xacro)
@@ -4,5 +4,5 @@
         <parent link="chassis"/>
         <child link="camera_link"/>
-        <origin xyz="0.0275 0 0.698" rpy="0 0 0"/>
+        <origin xyz="0.042 0 0.583" rpy="0 0 0"/>
     </joint>
     <link name="camera_link">

File: description/lidar.xacro (robot description, xacro)
@@ -2,7 +2,7 @@
 <robot xmlns:xacro="http://www.ros.org/wiki/xacro" >
     <joint name="laser_joint" type="fixed">
-        <parent link="chassis"/>
+        <parent link="camera_link"/>
         <child link="laser_frame"/>
-        <origin xyz="-0.02 0 0.7" rpy="0 0 0"/>
+        <origin xyz="-0.0475 0 0.022" rpy="0 0 0"/>
     </joint>
     <link name="laser_frame">
@@ -45,6 +45,6 @@
                 </scan>
                 <range>
-                    <min>0.1</min>
-                    <max>20</max>
+                    <min>0.06</min>
+                    <max>5.6</max>
                 </range>
             </ray>

File: description/robot_core.xacro (robot description, xacro)
@@ -3,12 +3,12 @@
     <xacro:include filename="inertial_macros.xacro"/>
     <xacro:property name="chassis_radius" value="0.20"/>
-    <xacro:property name="chassis_length" value="0.112"/>
-    <xacro:property name="chassis_height" value="0.08"/>
-    <xacro:property name="chassis_mass" value="1.0"/>
-    <xacro:property name="wheel_radius" value="0.033"/>
-    <xacro:property name="wheel_thickness" value="0.026"/>
+    <xacro:property name="chassis_length" value="0.111"/>
+    <xacro:property name="chassis_height" value="0.072"/>
+    <xacro:property name="chassis_mass" value="3.0"/>
+    <xacro:property name="wheel_radius" value="0.0325"/>
+    <xacro:property name="wheel_thickness" value="0.0255"/>
     <xacro:property name="wheel_mass" value="0.05"/>
     <xacro:property name="wheel_offset_x" value="0.0"/>
-    <xacro:property name="wheel_offset_y" value="0.17"/>
+    <xacro:property name="wheel_offset_y" value="0.1685"/>
     <xacro:property name="wheel_offset_z" value="${-chassis_height+wheel_radius}"/>
     <xacro:property name="caster_wheel_radius" value="0.02"/>

Commit message: edit camera and lidar parameters

File: description/camera.xacro (robot description, xacro)
@@ -3,8 +3,8 @@
     <joint name="camera_joint" type="fixed">
         <parent link="chassis"/>
-        <child link="camera_link"/>
+        <child link="camera_color_frame"/>
         <origin xyz="0.042 0 0.583" rpy="0 0 0"/>
     </joint>
-    <link name="camera_link">
+    <link name="camera_color_frame">
         <visual>
             <geometry>
@@ -22,10 +22,10 @@
     </link>
     <joint name="camera_optical_joint" type="fixed">
-        <parent link="camera_link"/>
-        <child link="camera_link_optical"/>
+        <parent link="camera_color_frame"/>
+        <child link="camera_color_optical_frame"/>
         <origin xyz="0 0 0" rpy="${-pi/2} 0 ${-pi/2}"/>
     </joint>
-    <link name="camera_link_optical"></link>
-    <gazebo reference="camera_link">
+    <link name="camera_color_optical_frame"></link>
+    <gazebo reference="camera_color_frame">
         <material>Gazebo/White</material>
         <sensor name="camera" type="camera">

File: description/depth_camera.xacro (robot description, xacro)
@@ -3,8 +3,8 @@
     <joint name="camera_joint" type="fixed">
         <parent link="chassis"/>
-        <child link="camera_link"/>
+        <child link="camera_color_frame"/>
         <origin xyz="0.042 0 0.583" rpy="0 0 0"/>
     </joint>
-    <link name="camera_link">
+    <link name="camera_color_frame">
         <visual>
             <geometry>
@@ -22,10 +22,10 @@
     </link>
     <joint name="camera_optical_joint" type="fixed">
-        <parent link="camera_link"/>
-        <child link="camera_link_optical"/>
+        <parent link="camera_color_frame"/>
+        <child link="camera_color_optical_frame"/>
         <origin xyz="0 0 0" rpy="${-pi/2} 0 ${-pi/2}"/>
     </joint>
-    <link name="camera_link_optical"></link>
-    <gazebo reference="camera_link">
+    <link name="camera_color_optical_frame"></link>
+    <gazebo reference="camera_color_frame">
         <material>Gazebo/White</material>
         <sensor name="camera" type="depth">

File: description/lidar.xacro (robot description, xacro)
@@ -2,7 +2,7 @@
 <robot xmlns:xacro="http://www.ros.org/wiki/xacro" >
     <joint name="laser_joint" type="fixed">
-        <parent link="camera_link"/>
+        <parent link="camera_color_frame"/>
         <child link="laser_frame"/>
-        <origin xyz="-0.0475 0 0.022" rpy="0 0 0"/>
+        <origin xyz="-0.0475 0 0.025" rpy="0 0 0"/>
     </joint>
     <link name="laser_frame">

Commit message: update params of robot

File: description/camera.xacro (robot description, xacro)
@@ -3,8 +3,8 @@
     <joint name="camera_joint" type="fixed">
         <parent link="chassis"/>
-        <child link="camera_link"/>
-        <origin xyz="0.0275 0 0.6" rpy="0 0 0"/>
+        <child link="camera_color_frame"/>
+        <origin xyz="0.042 0 0.583" rpy="0 0 0"/>
     </joint>
-    <link name="camera_link">
+    <link name="camera_color_frame">
         <visual>
             <geometry>
@@ -22,10 +22,10 @@
     </link>
     <joint name="camera_optical_joint" type="fixed">
-        <parent link="camera_link"/>
-        <child link="camera_link_optical"/>
+        <parent link="camera_color_frame"/>
+        <child link="camera_color_optical_frame"/>
         <origin xyz="0 0 0" rpy="${-pi/2} 0 ${-pi/2}"/>
     </joint>
-    <link name="camera_link_optical"></link>
-    <gazebo reference="camera_link">
+    <link name="camera_color_optical_frame"></link>
+    <gazebo reference="camera_color_frame">
         <material>Gazebo/White</material>
         <sensor name="camera" type="camera">

File: description/depth_camera.xacro (robot description, xacro)
@@ -3,8 +3,8 @@
     <joint name="camera_joint" type="fixed">
         <parent link="chassis"/>
-        <child link="camera_link"/>
-        <origin xyz="0.0275 0 0.6" rpy="0 0 0"/>
+        <child link="camera_color_frame"/>
+        <origin xyz="0.042 0 0.583" rpy="0 0 0"/>
     </joint>
-    <link name="camera_link">
+    <link name="camera_color_frame">
         <visual>
             <geometry>
@@ -22,10 +22,10 @@
     </link>
     <joint name="camera_optical_joint" type="fixed">
-        <parent link="camera_link"/>
-        <child link="camera_link_optical"/>
+        <parent link="camera_color_frame"/>
+        <child link="camera_color_optical_frame"/>
         <origin xyz="0 0 0" rpy="${-pi/2} 0 ${-pi/2}"/>
     </joint>
-    <link name="camera_link_optical"></link>
-    <gazebo reference="camera_link">
+    <link name="camera_color_optical_frame"></link>
+    <gazebo reference="camera_color_frame">
         <material>Gazebo/White</material>
         <sensor name="camera" type="depth">

File: description/gazebo_control.xacro (robot description, xacro)
@@ -9,6 +9,6 @@
             <left_joint>left_wheel_joint</left_joint>
             <right_joint>right_wheel_joint</right_joint>
-            <wheel_separation>0.297</wheel_separation>
-            <wheel_diameter>0.066</wheel_diameter>
+            <wheel_separation>0.337</wheel_separation>
+            <wheel_diameter>0.065</wheel_diameter>
             <!-- Limits -->
             <max_wheel_torque>200</max_wheel_torque>

File: description/lidar.xacro (robot description, xacro)
@@ -2,5 +2,5 @@
 <robot xmlns:xacro="http://www.ros.org/wiki/xacro" >
     <joint name="laser_joint" type="fixed">
-        <parent link="camera_link"/>
+        <parent link="camera_color_frame"/>
         <child link="laser_frame"/>
         <origin xyz="-0.0475 0 0.022" rpy="0 0 0"/>
@@ -45,6 +45,6 @@
                 </scan>
                 <range>
-                    <min>0.1</min>
-                    <max>20</max>
+                    <min>0.06</min>
+                    <max>5.6</max>
                 </range>
             </ray>

File: description/ros2_control.xacro (robot description, xacro)
@@ -41,6 +41,6 @@
                     <param name="max">10</param>
                 </command_interface>
+                <state_interface name="position"/>
                 <state_interface name="velocity"/>
-                <state_interface name="position"/>
             </joint>
             <joint name="right_wheel_joint">
@@ -49,6 +49,6 @@
                     <param name="max">10</param>
                 </command_interface>
+                <state_interface name="position"/>
                 <state_interface name="velocity"/>
-                <state_interface name="position"/>
             </joint>
         </ros2_control>

Commit message: udpate param of calib camera and lidar

File: description/camera.xacro (robot description, xacro)
@@ -4,5 +4,5 @@
         <parent link="chassis"/>
         <child link="camera_color_frame"/>
-        <origin xyz="0.042 0 0.583" rpy="0 0 0"/>
+        <origin xyz="0.042 0 0.878" rpy="0 0 0"/>
     </joint>
     <link name="camera_color_frame">

File: description/lidar.xacro (robot description, xacro)
@@ -4,5 +4,5 @@
         <parent link="camera_color_frame"/>
         <child link="laser_frame"/>
-        <origin xyz="-0.0475 0 0.025" rpy="0 0.03844 -0.06579"/>
+        <origin xyz="-0.0475 0 0.025" rpy="0 0.03844 -0.041866"/>
     </joint>
     <link name="laser_frame">

File: description/ros2_control.xacro (robot description, xacro)
@@ -7,5 +7,5 @@
                 <param name="left_wheel_name">left_wheel_joint</param>
                 <param name="right_wheel_name">right_wheel_joint</param>
-                <param name="loop_rate">33.3333</param>
+                <param name="loop_rate">20</param>
                 <param name="device">/dev/ttyTHS1</param>
                 <param name="baud_rate">115200</param>
