Commit message: fix origin of params

File: description/depth_camera.xacro (robot description, xacro)
@@ -4,5 +4,5 @@
         <parent link="chassis"/>
         <child link="camera_color_frame"/>
-        <origin xyz="0.042 0 0.583" rpy="0 0 0"/>
+        <origin xyz="0.042 0 0.613" rpy="0 -0.03844 0"/>
     </joint>
     <link name="camera_color_frame">

File: description/lidar.xacro (robot description, xacro)
@@ -4,5 +4,5 @@
         <parent link="camera_color_frame"/>
         <child link="laser_frame"/>
-        <origin xyz="-0.0475 0 0.025" rpy="0 0 0"/>
+        <origin xyz="-0.0475 0 0.025" rpy="0 0.03844 -0.06579"/>
     </joint>
     <link name="laser_frame">

Commit message: update params of robot

File: description/depth_camera.xacro (robot description, xacro)
@@ -2,7 +2,7 @@
 <robot xmlns:xacro="http://www.ros.org/wiki/xacro" >
     <joint name="camera_joint" type="fixed">
-        <parent link="chassis"/>
+        <parent link="holder"/>
         <child link="camera_color_frame"/>
-        <origin xyz="0.042 0 0.613" rpy="0 -0.03844 0"/>
+        <origin xyz="0.042 0 0.03" rpy="0 -0.03844 0"/>
     </joint>
     <link name="camera_color_frame">

File: description/robot_core.xacro (robot description, xacro)
@@ -3,7 +3,14 @@
     <xacro:include filename="inertial_macros.xacro"/>
     <xacro:property name="chassis_radius" value="0.20"/>
-    <xacro:property name="chassis_length" value="0.111"/>
+    <xacro:property name="chassis_length" value="0.112"/>
     <xacro:property name="chassis_height" value="0.072"/>
-    <xacro:property name="chassis_mass" value="3.0"/>
+    <xacro:property name="chassis_mass" value="2.0"/>
+    <xacro:property name="tripod_radius" value="0.0115"/>
+    <xacro:property name="tripod_length" value="0.441"/>
+    <xacro:property name="tripod_mass" value="1.0"/>
+    <xacro:property name="holder_length" value="0.17"/>
+    <xacro:property name="holder_width" value="0.17"/>
+    <xacro:property name="holder_height" value="0.003"/>
+    <xacro:property name="holder_mass" value="0.1"/>
     <xacro:property name="wheel_radius" value="0.03185"/>
     <xacro:property name="wheel_thickness" value="0.0255"/>
@@ -11,5 +18,5 @@
     <xacro:property name="wheel_offset_x" value="0.0"/>
     <xacro:property name="wheel_offset_y" value="0.164"/>
-    <xacro:property name="wheel_offset_z" value="${-chassis_height+wheel_radius}"/>
+    <xacro:property name="wheel_offset_z" value="${-chassis_height-chassis_length/2+wheel_radius}"/>
     <xacro:property name="caster_wheel_radius" value="0.02"/>
     <xacro:property name="caster_wheel_mass" value="0.04"/>
@@ -46,9 +53,9 @@
         <parent link="base_link"/>
         <child link="chassis"/>
-        <origin xyz="0 0 0"/>
+        <origin xyz="0 0 ${chassis_height+chassis_length/2}"/>
     </joint>
     <link name="chassis">
         <visual>
-            <origin xyz = "0 0 ${chassis_length/2}"/>
+            <origin xyz = "0 0 0}"/>
             <geometry>
                 <cylinder length="${chassis_length}" radius="${chassis_radius}"/>
@@ -69,7 +76,61 @@
         <material>Gazebo/Orange</material>
     </gazebo>
+    <!-- TRIPOD -->
+    <joint name="tripod_joint" type="fixed">
+        <parent link="chassis"/>
+        <child link="tripod"/>
+        <origin xyz="0 0 ${chassis_height/2}"/>
+    </joint>
+    <link name="tripod">
+        <visual>
+            <origin xyz = "0 0 ${tripod_length/2}"/>
+            <geometry>
+                <cylinder length="${tripod_length}" radius="${tripod_radius}"/>
+            </geometry>
+            <material name="black"/>
+        </visual>
+        <collision>
+            <origin xyz = "0 0 ${tripod_length/2}"/>
+            <geometry>
+                <cylinder length="${tripod_length}" radius="${tripod_radius}"/>
+            </geometry>
+        </collision>
+        <xacro:inertial_cylinder mass="${tripod_mass}" length="${tripod_length}" radius="${tripod_radius}">
+            <origin xyz="0 0 ${tripod_length/2}" rpy="0 0 0"/>
+        </xacro:inertial_cylinder>
+    </link>
+    <gazebo reference="tripod">
+        <material>Gazebo/Black</material>
+    </gazebo>
+    <!-- HOLDER -->
+    <joint name="holder_joint" type="fixed">
+        <parent link="tripod"/>
+        <child link="holder"/>
+        <origin xyz="0 0 ${tripod_length}"/>
+    </joint>
+    <link name="holder">
+        <visual>
+            <origin xyz = "0 0 ${holder_height/2}"/>
+            <geometry>
+                <box size="${holder_length} ${holder_width} ${holder_height}"/>
+            </geometry>
+            <material name="blue"/>
+        </visual>
+        <collision>
+            <origin xyz = "0 0 ${holder_length/2}"/>
+            <geometry>
+                <box size="${holder_length} ${holder_width} ${holder_height}"/>
+            </geometry>
+        </collision>
+        <xacro:inertial_box mass="${holder_mass}" x="${holder_length}" y="${holder_width}" z="${holder_height}">
+            <origin xyz="${holder_length/2} 0 ${holder_height/2}" rpy="0 0 0"/>
+        </xacro:inertial_box>
+    </link>
+    <gazebo reference="holder">
+        <material>Gazebo/Blue</material>
+    </gazebo>
     <!-- LEFT WHEEL LINK -->
     <joint name="left_wheel_joint" type="continuous">
-        <parent link="base_link"/>
+        <parent link="chassis"/>
         <child link="left_wheel"/>
         <origin xyz="0 ${wheel_offset_y} ${wheel_offset_z}" rpy="-${pi/2} 0 0" />
@@ -97,5 +158,5 @@
     <!-- RIGHT WHEEL LINK -->
     <joint name="right_wheel_joint" type="continuous">
-        <parent link="base_link"/>
+        <parent link="chassis"/>
         <child link="right_wheel"/>
         <origin xyz="0 ${-wheel_offset_y} ${wheel_offset_z}" rpy="${pi/2} 0 0" />
