Commit message: update robot param

File: description/robot_core.xacro (robot description, xacro)
@@ -4,5 +4,4 @@
     <xacro:property name="chassis_radius" value="0.20"/>
     <xacro:property name="chassis_length" value="0.112"/>
-    <xacro:property name="chassis_width" value="0.265"/>
     <xacro:property name="chassis_height" value="0.08"/>
     <xacro:property name="chassis_mass" value="1.0"/>

Commit message: Update robot_core.xacro

File: description/robot_core.xacro (robot description, xacro)
@@ -57,5 +57,5 @@
     <link name="chassis">
         <visual>
-            <origin xyz = "0 0 0}"/>
+            <origin xyz = "0 0 0"/>
             <geometry>
                 <cylinder length="${chassis_length}" radius="${chassis_radius}"/>
